Commit message: changed pkg name

File: description/stopy.urdf (robot description, URDF)
Before this commit: robot stopy, 5 links, 4 joints
Links:
- link base_link: geometry collision mesh filename=package://patrolling_sim_ros2_gazebo/meshes/stopy_chull.stl; visual mesh filename=package://patrolling_sim_ros2_gazebo/meshes/stopy_decimated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
